File: Hardware/PcbArtiom.fsch v33.brd (EAGLE design)
At the start: 170.2 x 111.2 mm, 103 parts, among them IC1 BD5229G-TR, IC4 XC6220A331MR-G, J1 112A-TAAR-R03_ATTEND, J2 SAMACSYS_PARTS_USB4110-GF-A, J3 FH34SRJ-24S-0.5SH_99_, J4 QWIIC_RIGHT_ANGLE, Q1 20V/4.2A/52mΩ/1.4W, Q2 20V/4.2A/52mΩ/1.4W, Q3 SI1308EDL-T1-GE3, U1 W25Q512JVEIQ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

Commit message: Add files via upload
Parts:
- J3: value FH34SRJ-24S-0.5SH_99_ -> QWIIC_RIGHT_ANGLE; device DeskAssistant_v19_v1:FH34SRJ24S05SH99 -> DeskAssistant_v19_v1:JST04_1MM_RA
- J4: value QWIIC_RIGHT_ANGLE -> FH34SRJ-24S-0.5SH_99_; device DeskAssistant_v19_v1:JST04_1MM_RA -> DeskAssistant_v19_v1:FH34SRJ24S05SH99
- moved J3 82.7 mm to (165.1, 19.2), turned to 90 degrees
- moved J4 82.7 mm to (82.5, 14.0), turned to 0 degrees
- moved TP14 17.3 mm to (104.1, 59.7)
- moved TP13 12.8 mm to (81.3, 87.6)
- moved J2 0.31 mm to (167.3, 54.3)
Connections:
- removed net EPD_SC: U2.5
- net 3V3: now also J3.2; no longer J4.2
- net EPD_3V3: now also J4.15, J4.16; no longer J3.15, J3.16
- net EPD_BUSY: now also J4.9; no longer J3.9
- net EPD_CS: now also J4.12; no longer J3.12
- net EPD_DC: now also J4.11, U2.5; no longer J3.11
- net EPD_RST: now also J4.10; no longer J3.10
- net GDR: now also J4.2; no longer J3.2
- net GND: now also J3.1, J4.17, J4.8, J4.MP1, J4.MP2; no longer J3.17, J3.8, J3.MP1, J3.MP2, J4.1
- net MOSI: now also J4.14; no longer J3.14
- net N$10: now also J4.5; no longer J3.5
- net N$12: now also J4.4; no longer J3.4
- net N$13: now also J4.18; no longer J3.18
- net N$14: now also J4.19; no longer J3.19
- net N$17: now also J4.20; no longer J3.20
- net N$19: now also J4.22; no longer J3.22
- net N$21: now also J4.24; no longer J3.24
- net PREVGH: now also J4.21; no longer J3.21
- net PREVGL: now also J4.23; no longer J3.23
- net RESE: now also J4.3; no longer J3.3
- net SCK: now also J4.13; no longer J3.13
- net SCL: now also J3.4; no longer J4.4
- net SDA: now also J3.3; no longer J4.3
Routing:
- net EPD_DC: track 28.5 -> 110.7 mm
- net GND: track 121.7 -> 145.7 mm, vias 5 -> 32
- net VBUS: track 101.0 -> 119.7 mm
- net EPD_3V3_C: track 114.2 -> 127.5 mm
- net VUSB: track 33.3 -> 44.8 mm, vias 3 -> 2
- net DP: track 20.4 -> 30.9 mm
- net SDA: track 199.2 -> 202.4 mm
- net 3V3: track 458.3 -> 456.8 mm
- net N$11: track 20.3 -> 19.6 mm
Other:
- outline, holes or cut-outs redrawn

Commit message: Add files via upload
Routing:
- net RESET: track 129.8 -> 122.0 mm
- net EPD_CS: track 163.3 -> 156.3 mm
- net SDA: track 202.4 -> 197.4 mm
- net MISO: track 97.5 -> 95.8 mm
- net N$1: track 29.3 -> 30.5 mm
- net VBUS: track 119.7 -> 119.2 mm
